File: cansat-camera-pcb/connectorsection.kicad_sch (KiCad schematic)
At the start: 5 parts, among them J1 Conn_01x08_Pin, J4 Conn_02x10_Odd_Even, J5 Conn_02x10_Odd_Even

Commit message: Revert "Footprint assign"
This reverts commit b0d58344ac617605db2b6635d18d5284d5b3f755.
Parts:
- J1: footprint Connector_PinHeader_2.54mm:PinHeader_1x08_P2.54mm_Vertical -> (none)
- R4, R5: footprint Resistor_SMD:R_0201_0603Metric -> (none)
Changed lines of the file:
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@@
 			)
 		)
-		(property "Footprint" "Connector_PinHeader_2.54mm:PinHeader_1x08_P2.54mm_Vertical"
+		(property "Footprint" ""
 			(at 46.99 121.92 0)
 			(effects
@@
 			)
 		)
-		(property "Footprint" "Resistor_SMD:R_0201_0603Metric"
+		(property "Footprint" ""
 			(at 49.53 97.79 0)
 			(effects
@@
 			)
 		)
-		(property "Footprint" "Resistor_SMD:R_0201_0603Metric"
+		(property "Footprint" ""
 			(at 52.07 97.79 0)
 			(effects

Commit message: Footprint assign
Parts:
- J1: footprint (none) -> Connector_PinHeader_2.54mm:PinHeader_1x08_P2.54mm_Vertical
- R4, R5: footprint (none) -> Resistor_SMD:R_0201_0603Metric
Changed lines of the file:
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@@
 			)
 		)
-		(property "Footprint" ""
+		(property "Footprint" "Connector_PinHeader_2.54mm:PinHeader_1x08_P2.54mm_Vertical"
 			(at 46.99 121.92 0)
 			(effects
@@
 			)
 		)
-		(property "Footprint" ""
+		(property "Footprint" "Resistor_SMD:R_0201_0603Metric"
 			(at 49.53 97.79 0)
 			(effects
@@
 			)
 		)
-		(property "Footprint" ""
+		(property "Footprint" "Resistor_SMD:R_0201_0603Metric"
 			(at 52.07 97.79 0)
 			(effects
