File: cansat-camera-pcb/connectorsection.kicad_sch (KiCad schematic)
At the start: 5 parts, among them J1 Conn_01x08_Pin, J4 Conn_02x10_Odd_Even, J5 Conn_02x10_Odd_Even

Commit message: Alkatrész elhelyezés final
Parts:
- J1: footprint Connector_PinSocket_2.54mm:PinSocket_1x08_P2.54mm_Vertical -> Connector_PinHeader_2.54mm:PinHeader_1x08_P2.54mm_Vertical_SMD_Pin1Left
- J4, J5: footprint Connector_PinSocket_2.00mm:PinSocket_2x10_P2.00mm_Vertical -> Connector_PinHeader_2.00mm:PinHeader_2x10_P2.00mm_Vertical_SMD
Connections:
- net GND: now also J4.6 (Pin_6), J4.8 (Pin_8); no longer J4.7 (Pin_7), J4.9 (Pin_9)
- net OBC_I2C_1_SCL: now also J4.3 (Pin_3); no longer J4.4 (Pin_4)
- net OBC_I2C_1_SDA: now also J4.1 (Pin_1); no longer J4.2 (Pin_2)
- net OBC_I2C_2_SCL: now also J4.4 (Pin_4); no longer J4.3 (Pin_3)
- net OBC_I2C_2_SDA: now also J4.2 (Pin_2); no longer J4.1 (Pin_1)
- net OBC_UART_Rx: now also J4.16 (Pin_16); no longer J4.13 (Pin_13)
- net OBC_UART_Tx: now also J4.14 (Pin_14); no longer J4.11 (Pin_11)
Changed lines of the file:
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@@
-	)
-	(no_connect
-		(at 77.47 66.04)
 	)
 	(no_connect
@@
 	)
 	(no_connect
-		(at 77.47 63.5)
-	)
-	(no_connect
 		(at 121.92 53.34)
 	)
@@
 	)
 	(no_connect
+		(at 64.77 55.88)
+	)
+	(no_connect
 		(at 121.92 55.88)
 	)
@@
 	)
 	(no_connect
-		(at 77.47 55.88)
-	)
-	(no_connect
 		(at 64.77 53.34)
 	)
@@
 	)
 	(no_connect
-		(at 77.47 53.34)
+		(at 64.77 60.96)
 	)
 	(no_connect
@@
 	)
 	(no_connect
+		(at 64.77 63.5)
+	)
+	(no_connect
 		(at 109.22 55.88)
 	)
@@
 		(at 64.77 66.04)
 	)
+	(no_connect
+		(at 64.77 58.42)
+	)
 	(wire
 		(pts
@@
 	(wire
 		(pts
-			(xy 62.23 55.88) (xy 64.77 55.88)
+			(xy 80.01 53.34) (xy 77.47 53.34)
 		)
 		(stroke
@@
 	(wire
 		(pts
-			(xy 62.23 58.42) (xy 64.77 58.42)
-		)
-		(stroke
-			(width 0)
-			(type default)
-		)
-	)
-	(wire
-		(pts
 			(xy 39.37 115.57) (xy 39.37 116.84)
 		)
@@
 	(wire
 		(pts
+			(xy 80.01 55.88) (xy 77.47 55.88)
+		)
+		(stroke
+			(width 0)
+			(type default)
+		)
+	)
+	(wire
+		(pts
 			(xy 54.61 115.57) (xy 54.61 116.84)
 		)
@@
 		)
 	)
-	(hierarchical_label "OBC_UART_Tx"
-		(shape output)
-		(at 64.77 60.96 180)
+	(hierarchical_label "OBC_I2C_1_SDA"
+		(shape bidirectional)
+		(at 64.77 48.26 180)
 		(effects
 			(font
@@
 		)
 	)
-	(hierarchical_label "OBC_I2C_2_SDA"
+	(hierarchical_label "OBC_I2C_2_SCL"
 		(shape bidirectional)
-		(at 64.77 48.26 180)
+		(at 77.47 50.8 0)
 		(effects
 			(font
 				(size 1.27 1.27)
 			)
-			(justify right)
+			(justify left)
+		)
+	)
+	(hierarchical_label "OBC_UART_Tx"
+		(shape output)
+		(at 77.47 63.5 0)
+		(effects
+			(font
+				(size 1.27 1.27)
+			)
+			(justify left)
 		)
 	)
@@
 		)
 	)
-	(hierarchical_label "OBC_I2C_1_SDA"
-		(shape bidirectional)
-		(at 77.47 48.26 0)
-		(effects
-			(font
-				(size 1.27 1.27)
-			)
-			(justify left)
-		)
-	)
 	(hierarchical_label "UART_Tx"
 		(shape input)
@@
 		)
 	)
-	(hierarchical_label "OBC_I2C_2_SCL"
+	(hierarchical_label "OBC_I2C_2_SDA"
+		(shape bidirectional)
+		(at 77.47 48.26 0)
+		(effects
+			(font
+				(size 1.27 1.27)
+			)
+			(justify left)
+		)
+	)
+	(hierarchical_label "OBC_I2C_1_SCL"
 		(shape bidirectional)
 		(at 64.77 50.8 180)
@@
 		)
 	)
-	(hierarchical_label "OBC_I2C_1_SCL"
-		(shape bidirectional)
-		(at 77.47 50.8 0)
+	(hierarchical_label "OBC_UART_Rx"
+		(shape input)
+		(at 77.47 66.04 0)
 		(effects
 			(font
@@
 			)
 			(justify left)
-		)
-	)
-	(hierarchical_label "OBC_UART_Rx"
-		(shape input)
-		(at 64.77 63.5 180)
-		(effects
-			(font
-				(size 1.27 1.27)
-			)
-			(justify right)
 		)
 	)
@@
 			)
 		)
-		(property "Footprint" "Connector_PinSocket_2.00mm:PinSocket_2x10_P2.00mm_Vertical"
+		(property "Footprint" "Connector_PinHeader_2.00mm:PinHeader_2x10_P2.00mm_Vertical_SMD"
 			(at 69.85 58.42 0)
 			(effects
@@
 			)
 		)
-		(property "Footprint" "Connector_PinSocket_2.54mm:PinSocket_1x08_P2.54mm_Vertical"
+		(property "Footprint" "Connector_PinHeader_2.54mm:PinHeader_1x08_P2.54mm_Vertical_SMD_Pin1Left"
 			(at 46.99 121.92 0)
 			(effects
@@
 			)
 		)
-		(property "Footprint" "Connector_PinSocket_2.00mm:PinSocket_2x10_P2.00mm_Vertical"
+		(property "Footprint" "Connector_PinHeader_2.00mm:PinHeader_2x10_P2.00mm_Vertical_SMD"
 			(at 114.3 58.42 0)
 			(effects
@@
 	(symbol
 		(lib_id "power:GND")
-		(at 62.23 55.88 270)
+		(at 80.01 55.88 90)
 		(unit 1)
 		(exclude_from_sim no)
@@
 		(fields_autoplaced yes)
 		(property "Reference" "#PWR035"
-			(at 55.88 55.88 0)
+			(at 86.36 55.88 0)
 			(effects
 				(font
@@
 		)
 		(property "Value" "GND"
-			(at 58.42 55.8799 90)
+			(at 83.82 55.8801 90)
 			(effects
 				(font
@@
 		)
 		(property "Footprint" ""
-			(at 62.23 55.88 0)
+			(at 80.01 55.88 0)
 			(effects
 				(font
@@
 		)
 		(property "Datasheet" ""
-			(at 62.23 55.88 0)
+			(at 80.01 55.88 0)
 			(effects
 				(font
@@
 		)
 		(property "Description" "Power symbol creates a global label with name \"GND\" , ground"
-			(at 62.23 55.88 0)
+			(at 80.01 55.88 0)
 			(effects
 				(font
@@
 	(symbol
 		(lib_id "power:GND")
-		(at 62.23 58.42 270)
+		(at 80.01 53.34 90)
 		(unit 1)
 		(exclude_from_sim no)
@@
 		(fields_autoplaced yes)
 		(property "Reference" "#PWR036"
-			(at 55.88 58.42 0)
+			(at 86.36 53.34 0)
 			(effects
 				(font
@@
 		)
 		(property "Value" "GND"
-			(at 58.42 58.4199 90)
+			(at 83.82 53.3401 90)
 			(effects
 				(font
@@
 		)
 		(property "Footprint" ""
-			(at 62.23 58.42 0)
+			(at 80.01 53.34 0)
 			(effects
 				(font
@@
 		)
 		(property "Datasheet" ""
-			(at 62.23 58.42 0)
+			(at 80.01 53.34 0)
 			(effects
 				(font
@@
 		)
 		(property "Description" "Power symbol creates a global label with name \"GND\" , ground"
-			(at 62.23 58.42 0)
-			(effects
-				(font
+			(at 80.01 53.34 0)
+			(effects
+				(font

Commit message: ready
Parts:
- removed J1: Conn_01x08_Pin, Connector_PinHeader_2.54mm:PinHeader_1x08_P2.54mm_Vertical_SMD_Pin1Left, symbol Connector:Conn_01x08_Pin
- removed R4, R5: 10k, Capacitor_SMD:C_0402_1005Metric, symbol Device:R_Small
- added J3: Conn_01x05_Socket, gaia-camera-footprints:PinSocket_1x05_P2.54mm_Horizontal, symbol Connector:Conn_01x05_Socket
- added R12, R13: 10k, Resistor_SMD:R_0402_1005Metric, symbol Device:R_Small
Connections:
- net +3.3V: now also J3.1 (Pin_1), R12.2
- net BOOT0: now also J3.2 (Pin_2)
- net GND: now also J3.5 (Pin_5), R13.1
- net SWCLK: now also J3.3 (Pin_3), R13.2
- net SWDIO: now also J3.4 (Pin_4), R12.1
- net OBC_I2C_1_SCL: no longer names the net of J4.3 (Pin_3)
- net OBC_I2C_1_SDA: no longer names the net of J4.1 (Pin_1)
- net OBC_I2C_2_SCL: no longer names the net of J4.4 (Pin_4)
- net OBC_I2C_2_SDA: no longer names the net of J4.2 (Pin_2)
- no-connect marks 22 -> 26

Commit message: USB fix
Connections:
- net OBC_UART_Rx: now also J4.14 (Pin_14); no longer J4.16 (Pin_16)
- net OBC_UART_Tx: now also J4.12 (Pin_12); no longer J4.14 (Pin_14)
- net USB_DM: now reaches J4.15 (Pin_15)
- new net USB_DP: J4.16 (Pin_16)
- no-connect marks 26 -> 24
Changed lines of the file:
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@@
-	)
-	(no_connect
-		(at 77.47 60.96)
 	)
 	(no_connect
@@
 	)
 	(no_connect
-		(at 64.77 66.04)
-	)
-	(no_connect
 		(at 64.77 58.42)
 	)
@@
 		)
 	)
-	(hierarchical_label "OBC_UART_Tx"
-		(shape output)
+	(hierarchical_label "OBC_UART_Rx"
+		(shape input)
 		(at 77.47 63.5 0)
 		(effects
@@
 			)
 			(justify left)
+		)
+	)
+	(hierarchical_label "USB_DM"
+		(shape bidirectional)
+		(at 64.77 66.04 180)
+		(effects
+			(font
+				(size 1.27 1.27)
+			)
+			(justify right)
 		)
 	)
@@
 		)
 	)
+	(hierarchical_label "OBC_UART_Tx"
+		(shape output)
+		(at 77.47 60.96 0)
+		(effects
+			(font
+				(size 1.27 1.27)
+			)
+			(justify left)
+		)
+	)
+	(hierarchical_label "USB_DP"
+		(shape bidirectional)
+		(at 77.47 66.04 0)
+		(effects
+			(font
+				(size 1.27 1.27)
+			)
+			(justify left)
+		)
+	)
 	(hierarchical_label "SWCLK"
 		(shape bidirectional)
@@
 		(effects
 			(font
-				(size 1.27 1.27)
-			)
-			(justify left)
-		)
-	)
-	(hierarchical_label "OBC_UART_Rx"
-		(shape input)
-		(at 77.47 66.04 0)
-		(effects
-			(font

Commit message: sdcard deleted form this PCB
Connections:
- net USB_DM renamed usb_dn
- net USB_DP renamed usb_dp
Changed lines of the file:
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@@
 		)
 	)
-	(hierarchical_label "USB_DM"
+	(hierarchical_label "usb_dn"
 		(shape bidirectional)
 		(at 64.77 66.04 180)
@@
 		)
 	)
-	(hierarchical_label "USB_DP"
+	(hierarchical_label "usb_dp"
 		(shape bidirectional)
 		(at 77.47 66.04 0)

Commit message: -
Connections:
- net usb_dn renamed usb_DN
- net usb_dp renamed usb_DP
Changed lines of the file:
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@@
 		)
 	)
-	(hierarchical_label "usb_dn"
+	(hierarchical_label "usb_DN"
 		(shape bidirectional)
 		(at 64.77 66.04 180)
@@
 		)
 	)
-	(hierarchical_label "usb_dp"
+	(hierarchical_label "usb_DP"
 		(shape bidirectional)
 		(at 77.47 66.04 0)

Commit message: fixes
Connections:
- net pwrkey: now reaches J5.11 (Pin_11)
- net reset: now reaches J5.12 (Pin_12)
- no-connect marks 24 -> 22
Changed lines of the file:
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@@
-	)
-	(no_connect
-		(at 121.92 60.96)
 	)
 	(no_connect
@@
 	)
 	(no_connect
-		(at 109.22 60.96)
-	)
-	(no_connect
 		(at 121.92 53.34)
 	)
@@
 	(wire
 		(pts
+			(xy 121.92 60.96) (xy 123.19 60.96)
+		)
+		(stroke
+			(width 0)
+			(type default)
+		)
+	)
+	(wire
+		(pts
 			(xy 39.37 102.87) (xy 39.37 113.03)
 		)
@@
 	(wire
 		(pts
+			(xy 107.95 60.96) (xy 109.22 60.96)
+		)
+		(stroke
+			(width 0)
+			(type default)
+		)
+	)
+	(wire
+		(pts
 			(xy 36.83 109.22) (xy 35.56 109.22)
 		)
@@
 			(width 0)
 			(type default)
+		)
+	)
+	(hierarchical_label "reset"
+		(shape output)
+		(at 123.19 60.96 0)
+		(effects
+			(font
+				(size 1.27 1.27)
+			)
+			(justify left)
 		)
 	)
@@
 		(effects
 			(font
+				(size 1.27 1.27)
+			)
+			(justify right)
+		)
+	)
+	(hierarchical_label "pwrkey"
+		(shape output)
+		(at 107.95 60.96 180)
+		(effects
+			(font

Commit message: Camera_Final
Connections:
- net GND: now also J4.10 (Pin_10); no longer J4.6 (Pin_6)
- net I2C2_SDA: now reaches J4.1 (Pin_1)
- net I2C4_SDA: now reaches J4.2 (Pin_2)
- net I2C2_SCL: now reaches J4.3 (Pin_3)
- net I2C4_SCL: now reaches J4.4 (Pin_4)
- no-connect marks 22 -> 18
Changed lines of the file:
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@@
-	)
-	(no_connect
-		(at 77.47 58.42)
-	)
-	(no_connect
-		(at 64.77 50.8)
-	)
-	(no_connect
-		(at 64.77 48.26)
 	)
 	(no_connect
@@
 	)
 	(no_connect
-		(at 77.47 48.26)
-	)
-	(no_connect
 		(at 64.77 55.88)
 	)
@@
 	)
 	(no_connect
-		(at 77.47 50.8)
-	)
-	(no_connect
 		(at 109.22 71.12)
 	)
@@
 	(no_connect
 		(at 109.22 55.88)
+	)
+	(no_connect
+		(at 77.47 53.34)
 	)
 	(no_connect
@@
 	(wire
 		(pts
-			(xy 80.01 53.34) (xy 77.47 53.34)
+			(xy 41.91 102.87) (xy 41.91 113.03)
 		)
 		(stroke
@@
 	(wire
 		(pts
-			(xy 41.91 102.87) (xy 41.91 113.03)
+			(xy 121.92 60.96) (xy 123.19 60.96)
 		)
 		(stroke
@@
 	(wire
 		(pts
-			(xy 121.92 60.96) (xy 123.19 60.96)
+			(xy 39.37 102.87) (xy 39.37 113.03)
 		)
 		(stroke
@@
 	(wire
 		(pts
-			(xy 39.37 102.87) (xy 39.37 113.03)
+			(xy 41.91 95.25) (xy 41.91 96.52)
 		)
 		(stroke
@@
 	(wire
 		(pts
-			(xy 41.91 95.25) (xy 41.91 96.52)
+			(xy 107.95 60.96) (xy 109.22 60.96)
 		)
 		(stroke
@@
 	(wire
 		(pts
-			(xy 107.95 60.96) (xy 109.22 60.96)
+			(xy 36.83 109.22) (xy 35.56 109.22)
 		)
 		(stroke
@@
 	(wire
 		(pts
-			(xy 36.83 109.22) (xy 35.56 109.22)
+			(xy 39.37 96.52) (xy 39.37 88.9)
 		)
 		(stroke
@@
 	(wire
 		(pts
-			(xy 39.37 96.52) (xy 39.37 88.9)
-		)
-		(stroke
-			(width 0)
-			(type default)
-		)
-	)
-	(wire
-		(pts
 			(xy 39.37 101.6) (xy 39.37 102.87)
-		)
-		(stroke
-			(width 0)
-			(type default)
-		)
-	)
-	(wire
-		(pts
-			(xy 80.01 55.88) (xy 77.47 55.88)
 		)
 		(stroke
@@
 		)
 	)
+	(hierarchical_label "I2C4_SCL"
+		(shape bidirectional)
+		(at 77.47 50.8 0)
+		(effects
+			(font
+				(size 1.27 1.27)
+			)
+			(justify left)
+		)
+	)
+	(hierarchical_label "I2C2_SCL"
+		(shape bidirectional)
+		(at 64.77 50.8 180)
+		(effects
+			(font
+				(size 1.27 1.27)
+			)
+			(justify right)
+		)
+	)
 	(hierarchical_label "BOOT0"
 		(shape input)
@@
 		)
 	)
+	(hierarchical_label "I2C2_SDA"
+		(shape bidirectional)
+		(at 64.77 48.26 180)
+		(effects
+			(font
+				(size 1.27 1.27)
+			)
+			(justify right)
+		)
+	)
 	(hierarchical_label "usb_DP"
 		(shape bidirectional)
@@
 		)
 	)
+	(hierarchical_label "I2C4_SDA"
+		(shape bidirectional)
+		(at 77.47 48.26 0)
+		(effects
+			(font
+				(size 1.27 1.27)
+			)
+			(justify left)
+		)
+	)
 	(symbol
 		(lib_id "power:VCC")
@@
 	(symbol
 		(lib_id "power:GND")
-		(at 80.01 55.88 90)
+		(at 77.47 55.88 90)
 		(unit 1)
 		(exclude_from_sim no)
@@
 		(fields_autoplaced yes)
 		(property "Reference" "#PWR035"
-			(at 86.36 55.88 0)
+			(at 83.82 55.88 0)
 			(effects
 				(font
@@
 		)
 		(property "Value" "GND"
-			(at 83.82 55.8801 90)
+			(at 81.28 55.8801 90)
 			(effects
 				(font
@@
 		)
 		(property "Footprint" ""
-			(at 80.01 55.88 0)
+			(at 77.47 55.88 0)
 			(effects
 				(font
@@
 		)
 		(property "Datasheet" ""
-			(at 80.01 55.88 0)
+			(at 77.47 55.88 0)
 			(effects
 				(font
@@
 		)
 		(property "Description" "Power symbol creates a global label with name \"GND\" , ground"
-			(at 80.01 55.88 0)
+			(at 77.47 55.88 0)
 			(effects
 				(font
@@
 	(symbol
 		(lib_id "power:GND")
-		(at 80.01 53.34 90)
-		(unit 1)
-		(exclude_from_sim no)
-		(in_bom yes)
-		(on_board yes)
-		(dnp no)
-		(fields_autoplaced yes)
-		(property "Reference" "#PWR036"
-			(at 86.36 53.34 0)
-			(effects
-				(font
-					(size 1.27 1.27)
-				)
-				(hide yes)
-			)
-		)
-		(property "Value" "GND"
-			(at 83.82 53.3401 90)
-			(effects
-				(font
-					(size 1.27 1.27)
-				)
-				(justify right)
-			)
-		)
-		(property "Footprint" ""
-			(at 80.01 53.34 0)
-			(effects
-				(font
-					(size 1.27 1.27)
-				)
-				(hide yes)
-			)
-		)
-		(property "Datasheet" ""
-			(at 80.01 53.34 0)
-			(effects
-				(font
-					(size 1.27 1.27)
-				)
-				(hide yes)
-			)
-		)
-		(property "Description" "Power symbol creates a global label with name \"GND\" , ground"
-			(at 80.01 53.34 0)
-			(effects
-				(font
-					(size 1.27 1.27)
-				)
-				(hide yes)
-			)
-		)
-		(pin "1"
-		)
-		(instances
-			(project "cansat-camera-pcb"
-				(path "/ff55e53a-9379-43eb-9b08-9bace1f81889/57ec086e-7f36-42c3-890c-c3ddf337b5b8"
-					(reference "#PWR036")
-					(unit 1)
-				)
-			)
-		)
-	)
-	(symbol
-		(lib_id "power:GND")
 		(at 77.47 71.12 90)
 		(unit 1)
@@
 					(unit 1)
 				)
+			)
+		)
+	)
+	(symbol
+		(lib_id "power:GND")
+		(at 77.47 58.42 90)
+		(unit 1)
+		(exclude_from_sim no)
+		(in_bom yes)
+		(on_board yes)
+		(dnp no)
+		(fields_autoplaced yes)
+		(property "Reference" "#PWR025"
+			(at 83.82 58.42 0)
+			(effects
+				(font
+					(size 1.27 1.27)
+				)
+				(hide yes)
+			)
+		)
+		(property "Value" "GND"
+			(at 81.28 58.4201 90)
+			(effects
+				(font
+					(size 1.27 1.27)
+				)
+				(justify right)
+			)
+		)
+		(property "Footprint" ""
+			(at 77.47 58.42 0)
+			(effects
+				(font
+					(size 1.27 1.27)
+				)
+				(hide yes)
+			)
+		)
+		(property "Datasheet" ""
+			(at 77.47 58.42 0)
+			(effects
+				(font
+					(size 1.27 1.27)
+				)
+				(hide yes)
+			)
+		)
+		(property "Description" "Power symbol creates a global label with name \"GND\" , ground"
+			(at 77.47 58.42 0)
+			(effects
+				(font
+					(size 1.27 1.27)
+				)
+				(hide yes)
+			)
+		)
+		(pin "1"
+		)
+		(instances
+			(project "cansat-camera-pcb"
+				(path "/ff55e53a-9379-43eb-9b08-9bace1f81889/57ec086e-7f36-42c3-890c-c3ddf337b5b8"
+					(reference "#PWR025")
+					(unit 1)
+				)

Commit message: some fixes
Connections:
- net I2C4_SCL: no longer names the net of J4.4 (Pin_4)
- net I2C4_SDA: no longer names the net of J4.2 (Pin_2)
- no-connect marks 18 -> 20
Changed lines of the file:
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@@
+	)
+	(no_connect
+		(at 77.47 50.8)
 	)
 	(no_connect
@@
 	(no_connect
 		(at 64.77 63.5)
+	)
+	(no_connect
+		(at 77.47 48.26)
 	)
 	(no_connect
@@
 		)
 	)
-	(hierarchical_label "I2C4_SCL"
-		(shape bidirectional)
-		(at 77.47 50.8 0)
-		(effects
-			(font
-				(size 1.27 1.27)
-			)
-			(justify left)
-		)
-	)
 	(hierarchical_label "I2C2_SCL"
 		(shape bidirectional)
@@
 		(effects
 			(font
-				(size 1.27 1.27)
-			)
-			(justify left)
-		)
-	)
-	(hierarchical_label "I2C4_SDA"
-		(shape bidirectional)
-		(at 77.47 48.26 0)
-		(effects
-			(font
