File: cansat-camera-pcb/connectorsection.kicad_sch (KiCad schematic)
At the start: 5 parts, among them J3 Conn_01x05_Socket, J4 Conn_02x10_Odd_Even, J5 Conn_02x10_Odd_Even

Commit message: dagobert bácsi hegyekben a steksz
Parts:
- removed J3: Conn_01x05_Socket, gaia-camera-footprints:PinSocket_1x05_P2.54mm_Horizontal, symbol Connector:Conn_01x05_Socket
- removed R12, R13: 10k, Resistor_SMD:R_0402_1005Metric, symbol Device:R_Small
- added J1: Conn_01x08_Socket, gaia-camera-footprints:HDR-SMD_8P-P2.00-H-F-W9.2, symbol Connector:Conn_01x08_Socket
Connections:
- net +3.3V: now also J1.1 (Pin_1), J1.5 (Pin_5)
- net GND: now also J1.4 (Pin_4), J1.8 (Pin_8)
- net SWCLK: now also J1.6 (Pin_6)
- net SWDIO: now also J1.7 (Pin_7)
- net OBC_UART_Rx: no longer names the net of J4.14 (Pin_14)
- net OBC_UART_Tx: no longer names the net of J4.12 (Pin_12)
- new net DEBUG_UARTRX: J1.3 (Pin_3)
- new net DEBUG_UART_TX: J1.2 (Pin_2)
- no-connect marks 20 -> 22

Commit message: milan eszi a havat(unicummal)  (jonas is zabalja)
Connections:
- net DEBUG_UARTRX is gone; now on net DEBUG_UART_TX: J1.3 (Pin_3)
- net +3.3V: no longer J1.1 (Pin_1)
- net DEBUG_UART_TX: no longer J1.2 (Pin_2)
- net VCC: now also J1.1 (Pin_1)
- net usb_DN renamed USB_DN
- net usb_DP renamed USB_DP
- new net DEBUG_UART_RX: J1.2 (Pin_2)
Changed lines of the file:
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@@
+	(wire
+		(pts
+			(xy 78.74 66.04) (xy 77.47 66.04)
+		)
+		(stroke
+			(width 0)
+			(type default)
+		)
+	)
 	(wire
 		(pts
@@
 	(wire
 		(pts
-			(xy 107.95 60.96) (xy 109.22 60.96)
+			(xy 63.5 66.04) (xy 64.77 66.04)
 		)
 		(stroke
@@
 	(wire
 		(pts
-			(xy 52.07 105.41) (xy 52.07 114.3)
+			(xy 107.95 60.96) (xy 109.22 60.96)
 		)
 		(stroke
 			(width 0)
 			(type default)
+		)
+	)
+	(wire
+		(pts
+			(xy 52.07 105.41) (xy 52.07 114.3)
+		)
+		(stroke
+			(width 0)
+			(type default)
+		)
+	)
+	(global_label "USB_DP"
+		(shape bidirectional)
+		(at 78.74 66.04 0)
+		(fields_autoplaced yes)
+		(effects
+			(font
+				(size 1.27 1.27)
+			)
+			(justify left)
+		)
+		(property "Intersheetrefs" "${INTERSHEET_REFS}"
+			(at 90.1541 66.04 0)
+			(effects
+				(font
+					(size 1.27 1.27)
+				)
+				(justify left)
+				(hide yes)
+			)
+		)
+	)
+	(global_label "USB_DN"
+		(shape bidirectional)
+		(at 63.5 66.04 180)
+		(fields_autoplaced yes)
+		(effects
+			(font
+				(size 1.27 1.27)
+			)
+			(justify right)
+		)
+		(property "Intersheetrefs" "${INTERSHEET_REFS}"
+			(at 52.0254 66.04 0)
+			(effects
+				(font
+					(size 1.27 1.27)
+				)
+				(justify right)
+				(hide yes)
+			)
 		)
 	)
@@
 		)
 	)
-	(hierarchical_label "usb_DN"
-		(shape bidirectional)
-		(at 64.77 66.04 180)
-		(effects
-			(font
-				(size 1.27 1.27)
-			)
-			(justify right)
-		)
-	)
-	(hierarchical_label "DEBUG_UARTRX"
+	(hierarchical_label "DEBUG_UART_TX"
 		(shape output)
 		(at 49.53 105.41 90)
@@
 		)
 	)
-	(hierarchical_label "usb_DP"
-		(shape bidirectional)
-		(at 77.47 66.04 0)
-		(effects
-			(font
-				(size 1.27 1.27)
-			)
-			(justify left)
-		)
-	)
-	(hierarchical_label "DEBUG_UART_TX"
+	(hierarchical_label "DEBUG_UART_RX"
 		(shape input)
 		(at 52.07 105.41 90)
@@
 	)
 	(symbol
-		(lib_id "power:+3.3V")
-		(at 54.61 113.03 0)
-		(unit 1)
-		(exclude_from_sim no)
-		(in_bom yes)
-		(on_board yes)
-		(dnp no)
-		(property "Reference" "#PWR073"
-			(at 54.61 116.84 0)
-			(effects
-				(font
-					(size 1.27 1.27)
-				)
-				(hide yes)
-			)
-		)
-		(property "Value" "+3.3V"
-			(at 54.61 107.188 90)
-			(effects
-				(font
-					(size 1.27 1.27)
-				)
-			)
-		)
-		(property "Footprint" ""
-			(at 54.61 113.03 0)
-			(effects
-				(font
-					(size 1.27 1.27)
-				)
-				(hide yes)
-			)
-		)
-		(property "Datasheet" ""
-			(at 54.61 113.03 0)
-			(effects
-				(font
-					(size 1.27 1.27)
-				)
-				(hide yes)
-			)
-		)
-		(property "Description" "Power symbol creates a global label with name \"+3.3V\""
-			(at 54.61 113.03 0)
-			(effects
-				(font
-					(size 1.27 1.27)
-				)
-				(hide yes)
-			)
-		)
-		(pin "1"
-		)
-		(instances
-			(project "cansat-camera-pcb"
-				(path "/ff55e53a-9379-43eb-9b08-9bace1f81889/57ec086e-7f36-42c3-890c-c3ddf337b5b8"
-					(reference "#PWR073")
-					(unit 1)
-				)
-			)
-		)
-	)
-	(symbol
 		(lib_id "Connector_Generic:Conn_02x10_Odd_Even")
 		(at 114.3 58.42 0)
@@
 					(unit 1)
 				)
+			)
+		)
+	)
+	(symbol
+		(lib_id "power:VCC")
+		(at 54.61 113.03 0)
+		(unit 1)
+		(exclude_from_sim no)
+		(in_bom yes)
+		(on_board yes)
+		(dnp no)
+		(property "Reference" "#PWR09"
+			(at 54.61 116.84 0)
+			(effects
+				(font
+					(size 1.27 1.27)
+				)
+				(hide yes)
+			)
+		)
+		(property "Value" "VCC"
+			(at 54.61 108.204 90)
+			(effects
+				(font
+					(size 1.27 1.27)
+				)
+			)
+		)
+		(property "Footprint" ""
+			(at 54.61 113.03 0)
+			(effects
+				(font
+					(size 1.27 1.27)
+				)
+				(hide yes)
+			)
+		)
+		(property "Datasheet" ""
+			(at 54.61 113.03 0)
+			(effects
+				(font
+					(size 1.27 1.27)
+				)
+				(hide yes)
+			)
+		)
+		(property "Description" "Power symbol creates a global label with name \"VCC\""
+			(at 54.61 113.03 0)
+			(effects
+				(font
+					(size 1.27 1.27)
+				)
+				(hide yes)
+			)
+		)
+		(pin "1"
+		)
+		(instances
+			(project "cansat-camera-pcb"
+				(path "/ff55e53a-9379-43eb-9b08-9bace1f81889/57ec086e-7f36-42c3-890c-c3ddf337b5b8"
+					(reference "#PWR09")
+					(unit 1)
+				)

Commit message: Update connectorsection.kicad_sch
Connections:
- net GND: now also J4.6 (Pin_6), J4.9 (Pin_9)
- no-connect marks 22 -> 20
Changed lines of the file:
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@@
 		(at 109.22 55.88)
-	)
-	(no_connect
-		(at 77.47 53.34)
-	)
-	(no_connect
-		(at 64.77 58.42)
 	)
 	(wire
@@
 	)
 	(symbol
+		(lib_id "power:GND")
+		(at 64.77 58.42 270)
+		(unit 1)
+		(exclude_from_sim no)
+		(in_bom yes)
+		(on_board yes)
+		(dnp no)
+		(fields_autoplaced yes)
+		(property "Reference" "#PWR099"
+			(at 58.42 58.42 0)
+			(effects
+				(font
+					(size 1.27 1.27)
+				)
+				(hide yes)
+			)
+		)
+		(property "Value" "GND"
+			(at 60.96 58.4199 90)
+			(effects
+				(font
+					(size 1.27 1.27)
+				)
+				(justify right)
+			)
+		)
+		(property "Footprint" ""
+			(at 64.77 58.42 0)
+			(effects
+				(font
+					(size 1.27 1.27)
+				)
+				(hide yes)
+			)
+		)
+		(property "Datasheet" ""
+			(at 64.77 58.42 0)
+			(effects
+				(font
+					(size 1.27 1.27)
+				)
+				(hide yes)
+			)
+		)
+		(property "Description" "Power symbol creates a global label with name \"GND\" , ground"
+			(at 64.77 58.42 0)
+			(effects
+				(font
+					(size 1.27 1.27)
+				)
+				(hide yes)
+			)
+		)
+		(pin "1"
+		)
+		(instances
+			(project "cansat-camera-pcb"
+				(path "/ff55e53a-9379-43eb-9b08-9bace1f81889/57ec086e-7f36-42c3-890c-c3ddf337b5b8"
+					(reference "#PWR099")
+					(unit 1)
+				)
+			)
+		)
+	)
+	(symbol
 		(lib_id "Connector_Generic:Conn_02x10_Odd_Even")
 		(at 114.3 58.42 0)
@@
 					(unit 1)
 				)
+			)
+		)
+	)
+	(symbol
+		(lib_id "power:GND")
+		(at 77.47 53.34 90)
+		(unit 1)
+		(exclude_from_sim no)
+		(in_bom yes)
+		(on_board yes)
+		(dnp no)
+		(fields_autoplaced yes)
+		(property "Reference" "#PWR098"
+			(at 83.82 53.34 0)
+			(effects
+				(font
+					(size 1.27 1.27)
+				)
+				(hide yes)
+			)
+		)
+		(property "Value" "GND"
+			(at 81.28 53.3401 90)
+			(effects
+				(font
+					(size 1.27 1.27)
+				)
+				(justify right)
+			)
+		)
+		(property "Footprint" ""
+			(at 77.47 53.34 0)
+			(effects
+				(font
+					(size 1.27 1.27)
+				)
+				(hide yes)
+			)
+		)
+		(property "Datasheet" ""
+			(at 77.47 53.34 0)
+			(effects
+				(font
+					(size 1.27 1.27)
+				)
+				(hide yes)
+			)
+		)
+		(property "Description" "Power symbol creates a global label with name \"GND\" , ground"
+			(at 77.47 53.34 0)
+			(effects
+				(font
+					(size 1.27 1.27)
+				)
+				(hide yes)
+			)
+		)
+		(pin "1"
+		)
+		(instances
+			(project "cansat-camera-pcb"
+				(path "/ff55e53a-9379-43eb-9b08-9bace1f81889/57ec086e-7f36-42c3-890c-c3ddf337b5b8"
+					(reference "#PWR098")
+					(unit 1)
+				)
