File: cansat-camera-pcb/cansat-camera-pcb.kicad_sch (KiCad schematic)
At the start: 25 parts, among them SW2 SW_Push, U4 STM32H743ZITx, Y1 24MHz

Commit message: send to production
Parts:
- U4: footprint Package_QFP:LQFP-144_20x20mm_P0.5mm -> gaia-camera-footprints:LQFP-144_20x20mm_P0.5mm
- Y1: footprint Crystal:Crystal_SMD_3225-4Pin_3.2x2.5mm -> gaia-camera-footprints:Crystal_SMD_3225-4Pin_3.2x2.5mm
Changed lines of the file:
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@@
 			)
 		)
-		(property "Footprint" "Package_QFP:LQFP-144_20x20mm_P0.5mm"
+		(property "Footprint" "gaia-camera-footprints:LQFP-144_20x20mm_P0.5mm"
 			(at 62.23 242.57 0)
 			(effects
@@
 			)
 		)
-		(property "Footprint" "Crystal:Crystal_SMD_3225-4Pin_3.2x2.5mm"
+		(property "Footprint" "gaia-camera-footprints:Crystal_SMD_3225-4Pin_3.2x2.5mm"
 			(at 44.45 91.44 0)
 			(effects

Commit message: dagobert bácsi hegyekben a steksz
Other:
- sheet Connector section ports: added DEBUG_UARTRX, DEBUG_UART_TX; removed BOOT0, OBC_UART_Rx, OBC_UART_Tx
Changed lines of the file:
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@@
 	(wire
 		(pts
-			(xy 193.04 170.18) (xy 190.5 170.18)
-		)
-		(stroke
-			(width 0)
-			(type default)
-		)
-	)
-	(wire
-		(pts
 			(xy 158.75 60.96) (xy 160.02 60.96)
 		)
@@
 	(wire
 		(pts
-			(xy 190.5 172.72) (xy 193.04 172.72)
+			(xy 190.5 171.45) (xy 193.04 171.45)
 		)
 		(stroke
@@
 	(wire
 		(pts
-			(xy 190.5 175.26) (xy 193.04 175.26)
+			(xy 190.5 173.99) (xy 193.04 173.99)
 		)
 		(stroke
@@
 	(wire
 		(pts
-			(xy 190.5 177.8) (xy 193.04 177.8)
+			(xy 190.5 176.53) (xy 193.04 176.53)
 		)
 		(stroke
@@
 	(wire
 		(pts
-			(xy 190.5 180.34) (xy 193.04 180.34)
+			(xy 190.5 179.07) (xy 193.04 179.07)
 		)
 		(stroke
@@
 	)
 	(label "LTE_reset"
-		(at 193.04 177.8 0)
+		(at 193.04 176.53 0)
 		(effects
 			(font
@@
 		)
 	)
-	(label "BOOT0"
-		(at 193.04 170.18 0)
-		(effects
-			(font
-				(size 1.27 1.27)
-			)
-			(justify left bottom)
-		)
-	)
 	(label "I2C4_SCL"
 		(at 156.21 181.61 180)
@@
 	)
 	(label "LTE_pwrkey"
-		(at 193.04 180.34 0)
+		(at 193.04 179.07 0)
 		(effects
 			(font
@@
 	)
 	(label "SWCLK"
-		(at 193.04 175.26 0)
+		(at 193.04 173.99 0)
 		(effects
 			(font
@@
 	)
 	(label "SWDIO"
-		(at 193.04 172.72 0)
+		(at 193.04 171.45 0)
 		(effects
 			(font
@@
 			)
 		)
-		(pin "BOOT0" input
-			(at 190.5 170.18 0)
-			(effects
-				(font
-					(size 1.27 1.27)
-				)
-				(justify right)
-			)
-		)
 		(pin "SWDIO" bidirectional
-			(at 190.5 172.72 0)
+			(at 190.5 171.45 0)
 			(effects
 				(font
@@
 		)
 		(pin "SWCLK" bidirectional
-			(at 190.5 175.26 0)
+			(at 190.5 173.99 0)
 			(effects
 				(font
@@
 			)
 		)
-		(pin "OBC_UART_Tx" output
-			(at 158.75 168.91 180)
-			(effects
-				(font
-					(size 1.27 1.27)
-				)
-				(justify left)
-			)
-		)
-		(pin "OBC_UART_Rx" input
-			(at 158.75 171.45 180)
-			(effects
-				(font
-					(size 1.27 1.27)
-				)
-				(justify left)
-			)
-		)
 		(pin "usb_DN" bidirectional
 			(at 158.75 176.53 180)
@@
 		)
 		(pin "reset" output
-			(at 190.5 177.8 0)
+			(at 190.5 176.53 0)
 			(effects
 				(font
@@
 		)
 		(pin "pwrkey" output
-			(at 190.5 180.34 0)
+			(at 190.5 179.07 0)
 			(effects
 				(font
@@
 			(effects
 				(font
+					(size 1.27 1.27)
+				)
+				(justify left)
+			)
+		)
+		(pin "DEBUG_UART_TX" input
+			(at 158.75 168.91 180)
+			(effects
+				(font
+					(size 1.27 1.27)
+				)
+				(justify left)
+			)
+		)
+		(pin "DEBUG_UARTRX" output
+			(at 158.75 171.45 180)
+			(effects
+				(font

Commit message: milan eszi a havat(unicummal)  (jonas is zabalja)
Parts:
- added R4, R5: 10k, Resistor_SMD:R_0402_1005Metric, symbol Device:R_Small
Connections:
- net DCMI_D2: now also U4.98 (PC8); no longer U4.125 (PG10)
- net DCMI_D3: now also U4.99 (PC9); no longer U4.126 (PG11)
- net LTE_pwrkey: now also U4.73 (PB12); no longer U4.2 (PE3)
- net LTE_reset: now also U4.74 (PB13); no longer U4.1 (PE2)
- net USART2_TX: now reaches U4.36 (PA2)
- net USART2_RX: now reaches U4.37 (PA3)
- net CAM_SCL: now reaches U4.69 (PB10)
- net CAM_SCL: now also R5.2
- net CAM_SDA: now reaches U4.70 (PB11)
- net CAM_SDA: now also R4.1
- net DCMI_HYSNC renamed DCMI_HSYNC
- net I2C4_SCL: no longer names the net of U4.81 (PD12)
- net I2C4_SDA: no longer names the net of U4.82 (PD13)
- net OV5640_PWDN renamed RCC_MCO_1
- net OV5640_RESET: no longer names the net of U4.101 (PA9)
- net UART4_RX: no longer names the net of U4.103 (PA11)
- net UART4_TX: no longer names the net of U4.104 (PA12)
- net usb_DN renamed USB_DN
- net usb_DP renamed USB_DP
- new net +3.3VA: R4.2, R5.1
- no-connect marks 50 -> 49
Other:
- sheet Connector section ports: added DEBUG_UART_RX; removed DEBUG_UARTRX, usb_DN, usb_DP
- sheet camera ports: added D2, D3, D4, D5, D6, D7, D8, D9, HSYNC, MCLK; removed DATA0, DATA1, DATA2, DATA3, DATA4, DATA5, DATA6, DATA7, DATA8, DATA9, HREF, PWDN, RESET, STROBE

Commit message: Finish
Vége
Parts:
- added D1: LED, LED_SMD:LED_0603_1608Metric, symbol Device:LED
- added R7: 1k, Resistor_SMD:R_0603_1608Metric, symbol Device:R_Small
Connections:
- net GND: now also R7.2
- net at U4.103 (PA11): now also D1.2 (A)
- new net: D1.1 (K), R7.1
- no-connect marks 49 -> 48
Changed lines of the file:
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@@
 	)
 	(no_connect
-		(at 123.19 97.79)
-	)
-	(no_connect
 		(at 123.19 120.65)
 	)
@@
 	(wire
 		(pts
+			(xy 134.62 97.79) (xy 135.89 97.79)
+		)
+		(stroke
+			(width 0)
+			(type default)
+		)
+	)
+	(wire
+		(pts
 			(xy 102.87 57.15) (xy 102.87 59.69)
 		)
@@
 	(wire
 		(pts
+			(xy 123.19 97.79) (xy 127 97.79)
+		)
+		(stroke
+			(width 0)
+			(type default)
+		)
+	)
+	(wire
+		(pts
 			(xy 172.72 53.34) (xy 173.99 53.34)
 		)
@@
 	)
 	(symbol
+		(lib_id "Device:LED")
+		(at 130.81 97.79 180)
+		(unit 1)
+		(exclude_from_sim no)
+		(in_bom yes)
+		(on_board yes)
+		(dnp no)
+		(property "Reference" "D1"
+			(at 130.81 92.456 0)
+			(effects
+				(font
+					(size 1.27 1.27)
+				)
+			)
+		)
+		(property "Value" "LED"
+			(at 130.81 94.742 0)
+			(effects
+				(font
+					(size 1.27 1.27)
+				)
+			)
+		)
+		(property "Footprint" "LED_SMD:LED_0603_1608Metric"
+			(at 130.81 97.79 0)
+			(effects
+				(font
+					(size 1.27 1.27)
+				)
+				(hide yes)
+			)
+		)
+		(property "Datasheet" "~"
+			(at 130.81 97.79 0)
+			(effects
+				(font
+					(size 1.27 1.27)
+				)
+				(hide yes)
+			)
+		)
+		(property "Description" "Light emitting diode"
+			(at 130.81 97.79 0)
+			(effects
+				(font
+					(size 1.27 1.27)
+				)
+				(hide yes)
+			)
+		)
+		(property "Sim.Pins" "1=K 2=A"
+			(at 130.81 97.79 0)
+			(effects
+				(font
+					(size 1.27 1.27)
+				)
+				(hide yes)
+			)
+		)
+		(pin "1"
+		)
+		(pin "2"
+		)
+		(instances
+			(project "cansat-camera-pcb"
+				(path "/ff55e53a-9379-43eb-9b08-9bace1f81889"
+					(reference "D1")
+					(unit 1)
+				)
+			)
+		)
+	)
+	(symbol
 		(lib_id "power:+3.3V")
 		(at 104.14 52.07 90)
@@
 	(symbol
 		(lib_id "power:GND")
+		(at 140.97 97.79 90)
+		(unit 1)
+		(exclude_from_sim no)
+		(in_bom yes)
+		(on_board yes)
+		(dnp no)
+		(fields_autoplaced yes)
+		(property "Reference" "#PWR097"
+			(at 147.32 97.79 0)
+			(effects
+				(font
+					(size 1.27 1.27)
+				)
+				(hide yes)
+			)
+		)
+		(property "Value" "GND"
+			(at 144.78 97.7899 90)
+			(effects
+				(font
+					(size 1.27 1.27)
+				)
+				(justify right)
+			)
+		)
+		(property "Footprint" ""
+			(at 140.97 97.79 0)
+			(effects
+				(font
+					(size 1.27 1.27)
+				)
+				(hide yes)
+			)
+		)
+		(property "Datasheet" ""
+			(at 140.97 97.79 0)
+			(effects
+				(font
+					(size 1.27 1.27)
+				)
+				(hide yes)
+			)
+		)
+		(property "Description" "Power symbol creates a global label with name \"GND\" , ground"
+			(at 140.97 97.79 0)
+			(effects
+				(font
+					(size 1.27 1.27)
+				)
+				(hide yes)
+			)
+		)
+		(pin "1"
+		)
+		(instances
+			(project ""
+				(path "/ff55e53a-9379-43eb-9b08-9bace1f81889"
+					(reference "#PWR097")
+					(unit 1)
+				)
+			)
+		)
+	)
+	(symbol
+		(lib_id "power:GND")
 		(at 57.15 85.09 270)
 		(unit 1)
@@
 					(unit 1)
 				)
+			)
+		)
+	)
+	(symbol
+		(lib_id "Device:R_Small")
+		(at 138.43 97.79 90)
+		(unit 1)
+		(exclude_from_sim no)
+		(in_bom yes)
+		(on_board yes)
+		(dnp no)
+		(fields_autoplaced yes)
+		(property "Reference" "R7"
+			(at 138.43 92.71 90)
+			(effects
+				(font
+					(size 1.016 1.016)
+				)
+			)
+		)
+		(property "Value" "1k"
+			(at 138.43 95.25 90)
+			(effects
+				(font
+					(size 1.27 1.27)
+				)
+			)
+		)
+		(property "Footprint" "Resistor_SMD:R_0603_1608Metric"
+			(at 138.43 97.79 0)
+			(effects
+				(font
+					(size 1.27 1.27)
+				)
+				(hide yes)
+			)
+		)
+		(property "Datasheet" "~"
+			(at 138.43 97.79 0)
+			(effects
+				(font
+					(size 1.27 1.27)
+				)
+				(hide yes)
+			)
+		)
+		(property "Description" "Resistor, small symbol"
+			(at 138.43 97.79 0)
+			(effects
+				(font
+					(size 1.27 1.27)
+				)
+				(hide yes)
+			)
+		)
+		(pin "1"
+		)
+		(pin "2"
+		)
+		(instances
+			(project "cansat-camera-pcb"
+				(path "/ff55e53a-9379-43eb-9b08-9bace1f81889"
+					(reference "R7")
+					(unit 1)
+				)
