File: cansat-camera-pcb/PSU.kicad_sch (KiCad schematic)
At the start: 3 parts, among them U2 AP2112K-3.3

Commit message: -
Parts:
- C14, C15: footprint Capacitor_SMD:C_0603_1608Metric -> (none)
- U2: footprint Package_TO_SOT_SMD:SOT-23-5 -> (none)
Changed lines of the file:
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@@
 			)
 		)
-		(property "Footprint" "Capacitor_SMD:C_0603_1608Metric"
+		(property "Footprint" ""
 			(at 85.09 60.96 0)
 			(effects
@@
 			)
 		)
-		(property "Footprint" "Package_TO_SOT_SMD:SOT-23-5"
+		(property "Footprint" ""
 			(at 96.52 60.325 0)
 			(effects
@@
 			)
 		)
-		(property "Footprint" "Capacitor_SMD:C_0603_1608Metric"
+		(property "Footprint" ""
 			(at 107.95 60.96 0)
 			(effects

Commit message: Footprint assign
Reset kivételével minden hozzácsatolva
Parts:
- C14, C15: footprint (none) -> Capacitor_SMD:C_0201_0603Metric
- U2: footprint (none) -> Package_TO_SOT_SMD:SOT-23-5_HandSoldering
Changed lines of the file:
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@@
 			)
 		)
-		(property "Footprint" ""
+		(property "Footprint" "Capacitor_SMD:C_0201_0603Metric"
 			(at 85.09 60.96 0)
 			(effects
@@
 			)
 		)
-		(property "Footprint" ""
+		(property "Footprint" "Package_TO_SOT_SMD:SOT-23-5_HandSoldering"
 			(at 96.52 60.325 0)
 			(effects
@@
 			)
 		)
-		(property "Footprint" ""
+		(property "Footprint" "Capacitor_SMD:C_0201_0603Metric"
 			(at 107.95 60.96 0)
 			(effects

Commit message: Footprint assign final
Parts:
- C14, C15: footprint Capacitor_SMD:C_0201_0603Metric -> Capacitor_SMD:C_0603_1608Metric
Changed lines of the file:
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@@
 			)
 		)
-		(property "Footprint" "Capacitor_SMD:C_0201_0603Metric"
+		(property "Footprint" "Capacitor_SMD:C_0603_1608Metric"
 			(at 85.09 60.96 0)
 			(effects
@@
 			)
 		)
-		(property "Footprint" "Capacitor_SMD:C_0201_0603Metric"
+		(property "Footprint" "Capacitor_SMD:C_0603_1608Metric"
 			(at 107.95 60.96 0)
 			(effects

Commit message: Regulator+
Parts:
- added C16, C17: 1uF, Capacitor_SMD:C_0603_1608Metric, symbol Device:C_Small
- added U1: AP2112K-3.3, Package_TO_SOT_SMD:SOT-23-5_HandSoldering, symbol Regulator_Linear:AP2112K-3.3
Connections:
- net GND: now also C16.2, C17.1, U1.2 (GND)
- net VCC: now also C16.1, U1.1 (VIN), U1.3 (EN)
- new net +3.3VA: C17.2, U1.5 (VOUT)
Other:
- moved on the sheet: C14, C15, U2

Commit message: send to production
Parts:
- U1, U2: footprint Package_TO_SOT_SMD:SOT-23-5_HandSoldering -> gaia-camera-footprints:SOT-23-5
Changed lines of the file:
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@@
 			)
 		)
-		(property "Footprint" "Package_TO_SOT_SMD:SOT-23-5_HandSoldering"
+		(property "Footprint" "gaia-camera-footprints:SOT-23-5"
 			(at 137.16 61.595 0)
 			(effects
@@
 			)
 		)
-		(property "Footprint" "Package_TO_SOT_SMD:SOT-23-5_HandSoldering"
+		(property "Footprint" "gaia-camera-footprints:SOT-23-5"
 			(at 73.66 61.595 0)
 			(effects

Commit message: milan eszi a havat(unicummal)  (jonas is zabalja)
Parts:
- added C23, C45, C46, C47, C49, C50: 10uF, Capacitor_SMD:C_0603_1608Metric, symbol Device:C_Small
- added C48, C6: 1uF, Capacitor_SMD:C_0603_1608Metric, symbol Device:C_Small
- added U3: TLV74315, gaia-camera-footprints:SOT-23-5, symbol gaia-camera-symbols:TLV74315
- added U5: TLV74328, gaia-camera-footprints:SOT-23-5, symbol gaia-camera-symbols:TLV74315
Connections:
- net +3.3VA: now also C23.2, C45.2, C46.2, C47.2, C48.2, C6.2, U3.1 (IN), U3.3 (EN), U5.1 (IN), U5.3 (EN)
- net GND: now also C23.1, C45.1, C46.1, C47.1, C48.1, C49.2, C50.2, C6.1, U3.2 (GND), U5.2 (GND)
- new net CAMERA_1.5V: C49.1, U5.5 (Vout)
- new net CAMERA_2.8V: C50.1, U3.5 (Vout)
Other:
- note added: "PSU"
- moved on the sheet: C14, C15, C16, C17, U1, U2

Commit message: OV5640 routing start
Parts:
- U3: value TLV74315 -> TLV74328
- U5: value TLV74328 -> TLV74315
Changed lines of the file:
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@@
 			)
 		)
-		(property "Value" "TLV74328"
+		(property "Value" "TLV74315"
 			(at 135.255 50.8 0)
 			(effects
@@
 			)
 		)
-		(property "Value" "TLV74315"
+		(property "Value" "TLV74328"
 			(at 135.255 26.67 0)
 			(effects
